Commit message: 20220113

File: my_ur_description/urdf/ur5/ur5_robot.urdf.xacro (robot description, xacro)
@@ -45,5 +45,5 @@
       <origin xyz="0 0 0.0" />
       <geometry>
-        <box size="1.1 0.7 0.03" />
+        <box size="0.7 1.1 0.03" />
       </geometry>
       <material name="LightGrey"/>
@@ -73,5 +73,5 @@
   </link>
   <joint name="mountingplate_joint" type="fixed">
-    <origin xyz="0.0 -0.20 0.021" />
+    <origin xyz="-0.2 0.0 0.021" />
     <parent link="baseplate_link" />
     <child link="mountingplate_link" />
@@ -81,5 +81,12 @@
     <parent link="mountingplate_link" />
     <child link="base_link" />
-    <origin xyz="0.0 0.0 0.01" rpy="0.0 0.0 ${-pi/2}"/>
+    <origin xyz="0.0 0.0 0.01" rpy="0.0 0.0 ${pi}"/>
+  </joint>
+  <!-- robot to mouting_plate. -->
+  <link name="tool_link" />
+  <joint name="tool0_link" type="fixed">
+    <parent link="tool0" />
+    <child link="tool_link" />
+    <origin xyz="0.0 0.0 0.0" rpy="0.0 ${pi} ${pi/2}"/>
   </joint>
 </robot>

Commit message: 20220114

File: my_ur_description/urdf/ur5/ur5_robot.urdf.xacro (robot description, xacro)
@@ -83,9 +83,9 @@
     <origin xyz="0.0 0.0 0.01" rpy="0.0 0.0 ${pi}"/>
   </joint>
-  <!-- robot to mouting_plate. -->
-  <link name="tool_link" />
+  <!-- tool center point -->
+  <link name="tcp_link" />
   <joint name="tool0_link" type="fixed">
     <parent link="tool0" />
-    <child link="tool_link" />
+    <child link="tcp_link" />
     <origin xyz="0.0 0.0 0.0" rpy="0.0 ${pi} ${pi/2}"/>
   </joint>

Commit message: 20220210

File: my_ur_description/urdf/ur5/ur5_robot.urdf.xacro (robot description, xacro)
@@ -14,6 +14,25 @@
     Refer to 'inc/ur_macro.xacro' for more information.
   -->
+<!--
+  <xacro:macro name="ur5_robot_system" params="
+   prefix
+   joint_limits_parameters_file:='$(find my_ur_description)/urdf/ur5/joint_limits.yaml'
+   kinematics_parameters_file:='$(find ur_description)/config/ur5/default_kinematics.yaml'
+   physical_parameters_file:='$(find ur_description)/config/ur5/physical_parameters.yaml'
+   visual_parameters_file:='$(find ur_description)/config/ur5/visual_parameters.yaml'
+   transmission_hw_interface:=hardware_interface/PositionJointInterface
+   safety_limits:=false
+   safety_pos_margin:=0.15
+   safety_k_position:=20
+   kinematics_config:='$(find ur_description)/config/ur5/default_kinematics.yaml
+   "
+  >
+-->
   <xacro:include filename="$(find my_ur_description)/urdf/ur5/ur5_macro.xacro"/>
-  <xacro:ur5_robot prefix="" />
+<!--
+  <xacro:arg name="kinematics_parameters" default="$(find ur_description)/config/ur5_default.yaml"/>
+  <xacro:ur5_robot prefix="" kinematics_parameters_file="${load_yaml('$(arg kinematics_parameters)')}"/>
+-->
+<xacro:ur5_robot prefix=""/>
   <material name="LightGrey">
       <color rgba="0.7 0.7 0.7 1.0" />
@@ -90,3 +109,6 @@
     <origin xyz="0.0 0.0 0.0" rpy="0.0 ${pi} ${pi/2}"/>
   </joint>
+<!--
+</xacro:macro>
+-->
 </robot>

Commit message: 20220212

File: my_ur_description/urdf/ur5/ur5_robot.urdf.xacro (robot description, xacro)
@@ -1,38 +1,15 @@
 <?xml version="1.0"?>
 <robot xmlns:xacro="http://wiki.ros.org/xacro" name="ur5_robot">
-  <!--
-    This is a convenience top-level xacro which loads the macro for the UR5e
-    which defines the default values for the various "parameters files"
-    parameters for a UR5e.
-    This file is only useful when loading a stand-alone, completely isolated
-    robot with only default values for all parameters such as the kinematics,
-    visual and physical parameters and joint limits.
-    This file is not intended to be integrated into a larger scene or other
-    composite xacro.
-    Instead, xacro:include 'inc/ur5e_macro.xacro' and override the defaults
-    for the arguments to that macro.
-    Refer to 'inc/ur_macro.xacro' for more information.
-  -->
-<!--
-  <xacro:macro name="ur5_robot_system" params="
-   prefix
-   joint_limits_parameters_file:='$(find my_ur_description)/urdf/ur5/joint_limits.yaml'
-   kinematics_parameters_file:='$(find ur_description)/config/ur5/default_kinematics.yaml'
-   physical_parameters_file:='$(find ur_description)/config/ur5/physical_parameters.yaml'
-   visual_parameters_file:='$(find ur_description)/config/ur5/visual_parameters.yaml'
-   transmission_hw_interface:=hardware_interface/PositionJointInterface
-   safety_limits:=false
-   safety_pos_margin:=0.15
-   safety_k_position:=20
-   kinematics_config:='$(find ur_description)/config/ur5/default_kinematics.yaml
-   "
-  >
--->
-  <xacro:include filename="$(find my_ur_description)/urdf/ur5/ur5_macro.xacro"/>
-<!--
-  <xacro:arg name="kinematics_parameters" default="$(find ur_description)/config/ur5_default.yaml"/>
-  <xacro:ur5_robot prefix="" kinematics_parameters_file="${load_yaml('$(arg kinematics_parameters)')}"/>
--->
-<xacro:ur5_robot prefix=""/>
+  <xacro:include filename="$(find ur_description)/urdf/inc/ur5_macro.xacro"/>
+  <xacro:ur5_robot
+    prefix = ""
+    joint_limits_parameters_file='$(find my_ur_description)/urdf/ur5/joint_limits.yaml'
+    kinematics_parameters_file='$(find ur_description)/config/ur5/default_kinematics.yaml'
+    physical_parameters_file='$(find ur_description)/config/ur5/physical_parameters.yaml'
+    visual_parameters_file='$(find ur_description)/config/ur5/visual_parameters.yaml'
+    transmission_hw_interface='hardware_interface/PositionJointInterface'
+    safety_limits='false'
+    safety_pos_margin='0.15'
+    safety_k_position='20'/>
   <material name="LightGrey">
       <color rgba="0.7 0.7 0.7 1.0" />
@@ -109,6 +86,3 @@
     <origin xyz="0.0 0.0 0.0" rpy="0.0 ${pi} ${pi/2}"/>
   </joint>
-<!--
-</xacro:macro>
--->
 </robot>
