Commit message: 20220217

File: my_ur_description/urdf/ur3/ur3_robot.urdf.xacro (robot description, xacro)
@@ -84,5 +84,5 @@
     <parent link="tool0" />
     <child link="tcp_link" />
-    <origin xyz="0.0 0.0 0.0" rpy="0.0 ${pi} ${pi/2}"/>
+    <origin xyz="0.0 0.0 0.0" rpy="0.0 ${-pi/2} 0.0"/>
   </joint>
 </robot>

File: my_ur_description/urdf/ur5/ur5_robot.urdf.xacro (robot description, xacro)
@@ -84,5 +84,5 @@
     <parent link="tool0" />
     <child link="tcp_link" />
-    <origin xyz="0.0 0.0 0.0" rpy="0.0 ${pi} ${pi/2}"/>
+    <origin xyz="0.0 0.0 0.0" rpy="0.0 ${-pi/2} 0.0"/>
   </joint>
 </robot>

File: my_ur_description/urdf/ur5e/ur5e_robot.urdf.xacro (robot description, xacro)
@@ -84,5 +84,5 @@
     <parent link="tool0" />
     <child link="tcp_link" />
-    <origin xyz="0.0 0.0 0.0" rpy="0.0 ${pi} ${pi/2}"/>
+    <origin xyz="0.0 0.0 0.0" rpy="0.0 ${-pi/2} 0.0"/>
   </joint>
 </robot>

Commit message: 20240412

File: my_ur_description/urdf/ur3/ur3_robot.urdf.xacro (robot description, xacro)
@@ -49,4 +49,9 @@
       <xacro:box_inertia m="10" x="1.1" y="0.7" z="0.03"/>
     </inertial>
+    <collision>
+      <geometry>
+        <box size="1.1 0.7 0.03" />
+      </geometry>
+    </collision>
   </link>
   <joint name="baseplate_joint" type="fixed">
@@ -67,4 +72,9 @@
       <xacro:box_inertia m="1" x="0.3" y="0.3" z="0.012"/>
     </inertial>
+    <collision>
+      <geometry>
+        <box size="0.3 0.3 0.012" />
+      </geometry>
+    </collision>
   </link>
   <joint name="mountingplate_joint" type="fixed">

File: my_ur_description/urdf/ur5/ur5_robot.urdf.xacro (robot description, xacro)
@@ -49,4 +49,9 @@
       <xacro:box_inertia m="10" x="1.1" y="0.7" z="0.03"/>
     </inertial>
+    <collision>
+      <geometry>
+        <box size="1.1 0.7 0.03" />
+      </geometry>
+    </collision>
   </link>
   <joint name="baseplate_joint" type="fixed">
@@ -67,4 +72,9 @@
       <xacro:box_inertia m="1" x="0.3" y="0.3" z="0.012"/>
     </inertial>
+    <collision>
+      <geometry>
+        <box size="0.3 0.3 0.012" />
+      </geometry>
+    </collision>
   </link>
   <joint name="mountingplate_joint" type="fixed">

File: my_ur_description/urdf/ur5e/ur5e_robot.urdf.xacro (robot description, xacro)
@@ -49,4 +49,9 @@
       <xacro:box_inertia m="10" x="1.1" y="0.7" z="0.03"/>
     </inertial>
+    <collision>
+      <geometry>
+        <box size="1.1 0.7 0.03" />
+      </geometry>
+    </collision>
   </link>
   <joint name="baseplate_joint" type="fixed">
@@ -67,4 +72,9 @@
       <xacro:box_inertia m="1" x="0.3" y="0.3" z="0.012"/>
     </inertial>
+    <collision>
+      <geometry>
+        <box size="0.3 0.3 0.012" />
+      </geometry>
+    </collision>
   </link>
   <joint name="mountingplate_joint" type="fixed">
